File: simo.kicad_pcb (KiCad board)
At the start: 2 copper layers, 63 x 120 mm, 14 parts, among them J10 Conn_01x10_Female, J11 Conn_01x16_Female, J12 Conn_01x14_Female, J13 Conn_01x16_Female, J14 Conn_01x10_Female, J3 Conector_Memoria_Flash_EXT, J4 Conn_01x04_Female, J5 Conn_01x02_Female, J6 Conn_01x02_Female, J7 Conn_01x16_Female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

Commit message: se agregaron huellas de : memoria flash ext, debug_usb y conversor_dc_dc
Parts:
- removed J10, J14: Conn_01x10_Female, Connector_PinSocket_2.54mm:PinSocket_1x10_P2.54mm_Vertical
- removed J11, J13, J7, J9: Conn_01x16_Female, Connector_PinSocket_2.54mm:PinSocket_1x16_P2.54mm_Vertical
- removed J12, J8: Conn_01x14_Female, Connector_PinSocket_2.54mm:PinSocket_1x14_P2.54mm_Vertical
- removed J3: Conector_Memoria_Flash_EXT, Connector_PinSocket_2.54mm:PinSocket_1x06_P2.54mm_Vertical
- removed the REF** at (90.0, 55.0)
- added REF**: BATERIA, bluepill:bateria, F.Cu at (108.1, 65.8)
- added U2: flash_externa, bluepill:conector_flash_ext, F.Cu at (122.7, 147.4)
- added U3: bateria, bluepill:bateria, F.Cu at (558.9, 6.60)
- added U4: USB_DEBUG, bluepill:debug_usb, F.Cu at (116.2, 151.9)
- moved J4 72.6 mm to (174.8, 144.3)
- moved J5 72.6 mm to (179.4, 144.3)
- moved J6 64.3 mm to (160.0, 112.7)
- moved U1 27.0 mm to (95.1, 123.8)
Connections:
- U1 pad 19: /PB8 -> Net-(U1-Pad19)
- U1 pad 25: Net-(J6-Pad2) -> Net-(U1-Pad25)
- U1 pad 26: Net-(J6-Pad1) -> Net-(U1-Pad26)
